Commit message: updated urdf files

File: src/kitbot_urdf/urdf/kitbot_physics.urdf (robot description, URDF)
Before this commit: robot visual, 5 links, 4 joints
Links:
- link back_left_wheel: geometry collision cylinder length=0.0254 radius=0.0762; visual cylinder length=0.0254 radius=0.0762
- link back_right_wheel: geometry collision cylinder length=0.0254 radius=0.0762; visual cylinder length=0.0254 radius=0.0762
- link base_link: geometry collision box size=.8 .6 .1; visual box size=.8 .6 .1
- link front_left_wheel: geometry collision cylinder length=0.0254 radius=0.0762; visual cylinder length=0.0254 radius=0.0762
- link front_right_wheel: geometry collision cylinder length=0.0254 radius=0.0762; visual cylinder length=0.0254 radius=0.0762
